File: _autosave-mudkip-themed-chaser.kicad_pcb (KiCad board)
At the start: 2 copper layers, 58.5 x 57 mm, 20 parts, among them J1 Conn_01x02, U1 NE555P, U2 4017

Commit message: added silkscreens
Other:
- board text added: "no idea :("
Changed lines of the file:
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@@
 			(drillshape 0)
 			(scaleselection 1)
-			(outputdirectory "")
+			(outputdirectory "production/")
 		)
 	)
@@
 		(layer "Edge.Cuts")
 	)
+	(gr_text "no idea :("
+		(at 169 95.4 0)
+		(layer "B.SilkS")
+		(effects
+			(font
+				(size 1.5 1.5)
+				(thickness 0.375)
+				(bold yes)
+			)
+			(justify mirror)
+		)
+	)
 	(gr_text "10000x weak to\nwater"
